File: HARDWARE/remoteLAB/bluetooth.kicad_sch (KiCad schematic)
At the start: 0 parts

Commit message: added symbols for display connector and BT part, added usb device to ioc
Parts:
- added AE1: Antenna, RF_Antenna:STM-BLUE-NRG-antenna, symbol Device:Antenna
- added C100, C37: 150n, symbol Device:C
- added C33, C38: 10n, symbol Device:C_Small
- added C34: 100n, symbol Device:C_Small
- added C35: 1u, symbol Device:C_Small
- added C36, C99: 100p, symbol Device:C
- added C39, C41, C43, C97: 1u, symbol Device:C
- added C40, C42, C46, C98: 100n, symbol Device:C
- added C44, C47: 22p, symbol Device:C_Small
- added C45, C48: 15p, symbol Device:C_Small
- added C49, C50: 1.2p, Capacitor_SMD:C_0402_1005Metric, symbol Device:C_Small
- added IC1: BALF-NRG-02D3, RF_Mini-Circuits:BALFNRG02D3, symbol tmp:BALF-NRG-02D3
- added J2: Conn_01x02, symbol Connector_Generic:Conn_01x02
- added L1: 10uH, LED_SMD:LED_RGB_Lumex_SML-LXT0805SIUGUBW, symbol Device:L
- added L2: 2nH, Inductor_SMD:L_0402_1005Metric, symbol Device:L
- added L3: 0 Ohm SM/L_0402 TBD_0402, symbol Device:L
- added L4: 3.3nH, Inductor_SMD:L_0402_1005Metric, symbol Device:L
- added R38: 1k, symbol Device:R_Small
- added R39, R41, R42: 4k7, symbol Device:R_Small
- added R40: 1K, symbol Device:R_Small
- added U13: AP130-15Y, Package_TO_SOT_SMD:SOT-89-3, symbol Regulator_Linear:AP130-15Y
- added U7: BlueNRG-232NS, Package_QFP:QFN50P500X500X100-33N-D, symbol RFLiB:BlueNRG-232N
- added Y2: 32.768kHz, symbol Device:Crystal_Small
- added Y3: 32MHz, symbol Device:Crystal_Small
Connections:
- new net: C44.2, C47.1, L2.1
- new net: C47.2, U7.22 (SXTAL1), Y2.1
- new net: C45.2, U7.18 (FXTAL0), Y3.2
- new net: C49.1, IC1.A1 (SE), L4.1
- new net: C34.2, C35.2, L1.1, U7.27 (SMPSFILT2)
- new net: R41.2, U7.30 (DIO12)
- new net: C48.2, U7.17 (FXTAL1), Y3.1
- new net: L1.2, U7.26 (SMPSFILT1)
- new net: AE1.1 (A), C50.1, L4.2
- new net: R40.1, U7.29 (DIO13)
- new net: C44.1, U7.23 (SXTAL0), Y2.2
- new net: C48.1, L3.1
- new net: J2.1 (Pin_1), R38.2
- new net: IC1.B2 (RF1), U7.20 (RF1)
- new net: IC1.B1 (RF0), U7.21 (RF0)
- new net +3V3: C39.1, C40.1, C41.1, C42.1, C43.1, C46.1, C97.1, C98.1, L1.3, R38.1, R41.1, R42.1, U13.3 (VI), U7.19 (VBAT2), U7.24 (VBAT1), U7.6 (VBAT3)
- new net BOOT: C33.1, J2.2 (Pin_2), R39.1, U7.4 (DIO7/BOOT)
- new net BT_RSTN: C38.1, R42.2, U7.25 (RESETN)
- new net BT_RX: U7.3 (DIO8)
- new net BT_TX: U7.32 (DIO11)
- new net BT_VDD1V2: C100.1, C36.1, C37.1, C99.1, U13.1 (VO), U7.28 (VDD1V2)
- new net GND: C100.2, C33.2, C34.1, C35.1, C36.2, C37.2, C38.2, C39.2, C40.2, C41.2, C42.2, C43.2, C45.1, C46.2, C49.2, C50.2, C97.2, C98.2, C99.2, IC1.A2 (GND), L2.2, L3.2, R39.2, R40.2, U13.2 (GND), U7.11 (DIO1), U7.12 (DIO0), U7.15 (ADC1), U7.16 (ADC2), U7.31 (TEST), U7.33 (GND), U7.5 (DIO6), U7.7 (DIO5), U7.8 (DIO4)
- no-connect marks 0 -> 6
Other:
- note added: "Solder a 10u_0805 between 1-2 or a 0R0_0402 between 1-3"
