File: HARDWARE/remoteLAB/ethernet.kicad_sch (KiCad schematic)
At the start: 0 parts

Commit message: added symbols for display connector and BT part, added usb device to ioc
Parts:
- added C10: 10u, symbol Device:C_Small
- added C11, C18, C19, C8: 100n, symbol Device:C
- added C12: 10u, symbol Device:C_Polarized_Small_US
- added C20, C21: 100n, symbol Device:C_Small
- added C22, C23: 27p, symbol Device:C_Small
- added C9: 0.1u, symbol Device:C_Small
- added FB2: FerriteBead, symbol Device:FerriteBead
- added FB3: FerriteBead, symbol Device:FerriteBead_Small
- added J13: RJ45_Amphenol_RJMG1BD3B8K1ANR, Connector_RJ:RJ45_Amphenol_RJMG1BD3B8K1ANR, symbol Connector:RJ45_Amphenol_RJMG1BD3B8K1ANR
- added JP2: Jumper_2_Bridged, symbol Jumper:Jumper_2_Bridged
- added R30, R32: 330, symbol Device:R_Small
- added R33, R34, R35, R36: 49.9 1%, symbol Device:R_Small
- added R37: 2.32k 1%, symbol Device:R_Small
- added R43: 1k, symbol Device:R_Small
- added R44: 5M, symbol Device:R_Small
- added R59: 10k, symbol Device:R_Small
- added U8: ENC28J60x-SO, Package_SO:SOIC-28W_7.5x17.9mm_P1.27mm, symbol Interface_Ethernet:ENC28J60x-SO
- added Y1: 25MHz, symbol Device:Crystal_Small
Connections:
- new net: C23.2, R44.1, Y1.1
- new net: R44.2, U8.24 (OSC2)
- new net: C9.1, R33.2, R34.2
- new net: C10.1, U8.1 (VCAP)
- new net: J13.L1, R32.1
- new net: R37.1, U8.14 (RBIAS)
- new net: C22.2, U8.23 (OSC1), Y1.2
- new net: C20.1, C21.1, FB3.1, U8.25 (VDDOSC)
- new net: J13.L4, R30.1
- new net +3V3: C11.1, C12.1, C8.1, FB2.2, FB3.2, R43.1, R59.1, U8.20 (VDDPLL), U8.28 (VDD)
- new net CLK: U8.9 (~{CS})
- new net CS: U8.8 (SCK)
- new net ETH_AGND: C18.2, C19.2, C9.2, JP2.2 (B), U8.11 (VSSRX), U8.18 (VSSTX)
- new net ETH_LEDG: R30.2, U8.26 (LEDB)
- new net ETH_LEDY: R32.2, U8.27 (LEDA)
- new net ETH_RST: R43.2, U8.10 (~{RESET})
- new net ETH_VDDA: C18.1, C19.1, FB2.1, J13.R4 (TCT), R35.2, R36.2, U8.15 (VDDTX), U8.19 (VDDRX)
- new net Earth: J13.R8, J13.SH
- new net GND: C10.2, C11.2, C12.2, C20.2, C21.2, C22.1, C23.1, C8.2, J13.L2, J13.L3, JP2.1 (A), R37.2, U8.2 (VSS), U8.21 (VSSPLL), U8.22 (VSSOSC)
- new net RX+: J13.R3 (RD+), R33.1, U8.13 (TPIN+)
- new net RX-: J13.R6 (RD-), R34.1, U8.12 (TPIN-)
- new net SI: U8.7 (SI)
- new net SO: U8.6 (SO)
- new net TX+: J13.R1 (TD+), R35.1, U8.17 (TPOUT+)
- new net TX-: J13.R2 (TD-), R36.1, U8.16 (TPOUT-)
- new net nINT: R59.2, U8.4 (~{INT})
- no-connect marks 0 -> 3
Other:
- note added: "ethernet 10/100 Mbit so 100MHz max"
