File: HARDWARE/remoteLAB/TFT.kicad_sch (KiCad schematic)
At the start: 0 parts

Commit message: added symbols for display connector and BT part, added usb device to ioc
Parts:
- added J1: Conn_01x45, Connector_FFC-FPC:FH2345S03SHAW05, symbol Connector_Generic:Conn_01x45
- added R1: 250, symbol Device:R
- added R2, R3: 10k, symbol Device:R
- added R4, R5, R6, R7: 47, symbol Device:R_Small
Connections:
- new net: R2.2, R7.2
- new net +3V3: J1.10 (Pin_10), J1.42 (Pin_42), J1.44 (Pin_44), J1.9 (Pin_9), R2.1, R3.1
- new net +3V3LED: R1.2
- new net CSX: J1.12 (Pin_12), R7.1
- new net GND: J1.13 (Pin_13), J1.15 (Pin_15), J1.18 (Pin_18), J1.19 (Pin_19), J1.20 (Pin_20), J1.21 (Pin_21), J1.22 (Pin_22), J1.23 (Pin_23), J1.24 (Pin_24), J1.25 (Pin_25), J1.26 (Pin_26), J1.27 (Pin_27), J1.28 (Pin_28), J1.29 (Pin_29), J1.30 (Pin_30), J1.31 (Pin_31), J1.32 (Pin_32), J1.33 (Pin_33), J1.34 (Pin_34), J1.35 (Pin_35), J1.36 (Pin_36), J1.37 (Pin_37), J1.38 (Pin_38), J1.39 (Pin_39), J1.40 (Pin_40), J1.43 (Pin_43), J1.45 (Pin_45), J1.8 (Pin_8)
- new net GNDLED: J1.1 (Pin_1), J1.2 (Pin_2), J1.3 (Pin_3), J1.4 (Pin_4), J1.5 (Pin_5), J1.6 (Pin_6)
- new net LEDA: J1.7 (Pin_7), R1.1
- new net RESET: J1.41 (Pin_41), R3.2
- new net SDA: J1.16 (Pin_16), R5.1
- new net SDO: J1.17 (Pin_17), R6.1
- new net TE: J1.11 (Pin_11)
- new net WRX/SCL: J1.14 (Pin_14), R4.1
- no-connect marks 0 -> 1
Other:
- note added: "120mA"
